File: hw/LED_NMOS_Row_Matrix.kicad_sch (KiCad schematic)
At the start: 8 parts

Commit message: updated sheets information
Other:
- company: (none) -> Qingdao IotPi Information Technology Ltd.,
- title: (none) -> KiCad 2023 Shen Zhen Badge
Changed lines of the file:
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@@
 (kicad_sch (version 20230121) (generator eeschema)
   (paper "A4")
+  (title_block
+    (title "KiCad 2023 Shen Zhen Badge")
+    (date "2023-09-04")
+    (rev "1")
+    (company "Qingdao IotPi Information Technology Ltd.,")
+    (comment 1 "Designed by Yang Hongbo")
+  )
   (wire (pts (xy 105.41 68.58) (xy 105.41 60.96))
     (stroke (width 0) (type default))

Commit message: updated components LCSC (2N7002T)
Parts:
- Q? (x8): LCSC (none) -> C5224243; Vendor (none) -> ElecSuper(静芯微）; Vendor Model (none) -> 2N7002T
Changed lines of the file:
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@@
+      (effects (font (size 1.27 1.27)) hide)
+    )
+    (property "Description" "类型: N沟道 漏源电压(Vdss): 60V 连续漏极电流(Id): 300mA 功率(Pd): 200mW 导通电阻(RDS(on)@Vgs,Id):" (at 182.88 73.66 0)
+      (effects (font (size 1.27 1.27)) hide)
+    )
+    (property "LCSC" "C5224243" (at 182.88 73.66 0)
+      (effects (font (size 1.27 1.27)) hide)
+    )
+    (property "Vendor" "ElecSuper(静芯微）" (at 182.88 73.66 0)
+      (effects (font (size 1.27 1.27)) hide)
+    )
+    (property "Vendor Model" "2N7002T" (at 182.88 73.66 0)
       (effects (font (size 1.27 1.27)) hide)
     )
@@
       (effects (font (size 1.27 1.27)) hide)
     )
+    (property "Description" "类型: N沟道 漏源电压(Vdss): 60V 连续漏极电流(Id): 300mA 功率(Pd): 200mW 导通电阻(RDS(on)@Vgs,Id):" (at 182.88 135.89 0)
+      (effects (font (size 1.27 1.27)) hide)
+    )
+    (property "LCSC" "C5224243" (at 182.88 135.89 0)
+      (effects (font (size 1.27 1.27)) hide)
+    )
+    (property "Vendor" "ElecSuper(静芯微）" (at 182.88 135.89 0)
+      (effects (font (size 1.27 1.27)) hide)
+    )
+    (property "Vendor Model" "2N7002T" (at 182.88 135.89 0)
+      (effects (font (size 1.27 1.27)) hide)
+    )
     (pin "1")
     (pin "2")
@@
       (effects (font (size 1.27 1.27)) hide)
     )
+    (property "Description" "类型: N沟道 漏源电压(Vdss): 60V 连续漏极电流(Id): 300mA 功率(Pd): 200mW 导通电阻(RDS(on)@Vgs,Id):" (at 182.88 104.14 0)
+      (effects (font (size 1.27 1.27)) hide)
+    )
+    (property "LCSC" "C5224243" (at 182.88 104.14 0)
+      (effects (font (size 1.27 1.27)) hide)
+    )
+    (property "Vendor" "ElecSuper(静芯微）" (at 182.88 104.14 0)
+      (effects (font (size 1.27 1.27)) hide)
+    )
+    (property "Vendor Model" "2N7002T" (at 182.88 104.14 0)
+      (effects (font (size 1.27 1.27)) hide)
+    )
     (pin "1")
     (pin "2")
@@
       (effects (font (size 1.27 1.27)) hide)
     )
+    (property "Description" "类型: N沟道 漏源电压(Vdss): 60V 连续漏极电流(Id): 300mA 功率(Pd): 200mW 导通电阻(RDS(on)@Vgs,Id):" (at 102.87 135.89 0)
+      (effects (font (size 1.27 1.27)) hide)
+    )
+    (property "LCSC" "C5224243" (at 102.87 135.89 0)
+      (effects (font (size 1.27 1.27)) hide)
+    )
+    (property "Vendor" "ElecSuper(静芯微）" (at 102.87 135.89 0)
+      (effects (font (size 1.27 1.27)) hide)
+    )
+    (property "Vendor Model" "2N7002T" (at 102.87 135.89 0)
+      (effects (font (size 1.27 1.27)) hide)
+    )
     (pin "1")
     (pin "2")
@@
       (effects (font (size 1.27 1.27)) hide)
     )
+    (property "Description" "类型: N沟道 漏源电压(Vdss): 60V 连续漏极电流(Id): 300mA 功率(Pd): 200mW 导通电阻(RDS(on)@Vgs,Id):" (at 102.87 73.66 0)
+      (effects (font (size 1.27 1.27)) hide)
+    )
+    (property "LCSC" "C5224243" (at 102.87 73.66 0)
+      (effects (font (size 1.27 1.27)) hide)
+    )
+    (property "Vendor" "ElecSuper(静芯微）" (at 102.87 73.66 0)
+      (effects (font (size 1.27 1.27)) hide)
+    )
+    (property "Vendor Model" "2N7002T" (at 102.87 73.66 0)
+      (effects (font (size 1.27 1.27)) hide)
+    )
     (pin "1")
     (pin "2")
@@
       (effects (font (size 1.27 1.27)) hide)
     )
+    (property "Description" "类型: N沟道 漏源电压(Vdss): 60V 连续漏极电流(Id): 300mA 功率(Pd): 200mW 导通电阻(RDS(on)@Vgs,Id):" (at 182.88 43.18 0)
+      (effects (font (size 1.27 1.27)) hide)
+    )
+    (property "LCSC" "C5224243" (at 182.88 43.18 0)
+      (effects (font (size 1.27 1.27)) hide)
+    )
+    (property "Vendor" "ElecSuper(静芯微）" (at 182.88 43.18 0)
+      (effects (font (size 1.27 1.27)) hide)
+    )
+    (property "Vendor Model" "2N7002T" (at 182.88 43.18 0)
+      (effects (font (size 1.27 1.27)) hide)
+    )
     (pin "1")
     (pin "2")
@@
       (effects (font (size 1.27 1.27)) hide)
     )
+    (property "Description" "类型: N沟道 漏源电压(Vdss): 60V 连续漏极电流(Id): 300mA 功率(Pd): 200mW 导通电阻(RDS(on)@Vgs,Id):" (at 102.87 43.18 0)
+      (effects (font (size 1.27 1.27)) hide)
+    )
+    (property "LCSC" "C5224243" (at 102.87 43.18 0)
+      (effects (font (size 1.27 1.27)) hide)
+    )
+    (property "Vendor" "ElecSuper(静芯微）" (at 102.87 43.18 0)
+      (effects (font (size 1.27 1.27)) hide)
+    )
+    (property "Vendor Model" "2N7002T" (at 102.87 43.18 0)
+      (effects (font (size 1.27 1.27)) hide)
+    )
     (pin "1")
     (pin "2")
@@
       (effects (font (size 1.27 1.27)) hide)
     )
+    (property "Description" "类型: N沟道 漏源电压(Vdss): 60V 连续漏极电流(Id): 300mA 功率(Pd): 200mW 导通电阻(RDS(on)@Vgs,Id):" (at 102.87 104.14 0)
+      (effects (font (size 1.27 1.27)) hide)
+    )
+    (property "LCSC" "C5224243" (at 102.87 104.14 0)
+      (effects (font (size 1.27 1.27)) hide)
+    )
+    (property "Vendor" "ElecSuper(静芯微）" (at 102.87 104.14 0)
+      (effects (font (size 1.27 1.27)) hide)
+    )
+    (property "Vendor Model" "2N7002T" (at 102.87 104.14 0)
+      (effects (font (size 1.27 1.27)) hide)
+    )
