File: hw/AP3410.kicad_sch (KiCad schematic)
At the start: 6 parts, among them U4 AP3410K

Commit message: updated sheets information
Other:
- company: (none) -> Qingdao IotPi Information Technology Ltd.,
- title: (none) -> KiCad 2023 Shen Zhen Badge
Changed lines of the file:
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@@
 (kicad_sch (version 20230121) (generator eeschema)
   (paper "A4")
+  (title_block
+    (title "KiCad 2023 Shen Zhen Badge")
+    (date "2023-09-04")
+    (rev "1")
+    (company "Qingdao IotPi Information Technology Ltd.,")
+    (comment 1 "Designed by Yang Hongbo")
+  )
   (junction (at 168.91 66.04) (diameter 0) (color 0 0 0 0)
   )
