File: hw/RGB_LED_Cell2.kicad_sch (KiCad schematic)
At the start: 4 parts

Commit message: changed Hardware design
Parts:
- removed D16: MHT151RGBCT, IotPi_LED:MeiHua_RGB_LED_Reverse_Mounting_MHT151RGBCT, symbol Device:LED_ABGR
- added D2: XL-1615RGBC-RF, IotPi_LED:XL-1615RGBC, symbol Device:LED_RGAB
- renumbered R46 to R7, R47 to R8, R48 to R9
Connections:
- net HighSide_Input: now also D2.3 (A)
- net at R7.1: now also D2.1 (RK)
- net at R9.1: now also D2.4 (BK)
- net at R8.1: now also D2.2 (GK)
