File: hw/RGB_LED_Cell2.kicad_sch (KiCad schematic)
At the start: 5 parts, among them Q15 SK2302AAT

Commit message: filled in LCSC
Parts:
- D2: LCSC (none) -> PH0094078
Changed lines of the file:
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@@
+      (effects (font (size 1.27 1.27)) hide)
+    )
+    (property "LCSC" "PH0094078" (at 147.32 86.36 0)
       (effects (font (size 1.27 1.27)) hide)
     )
