File: hw/LED_Row.kicad_sch (KiCad schematic)
At the start: 3 parts, among them Q2 SK2302AAT, Q3 SK2302AAT, Q4 SK2302AAT

Commit message: updated Sheet and Board Information
Other:
- company: (none) -> Beijing Exponential Deep Space
- title: (none) -> KiCad 2023 Asia Badge
Changed lines of the file:
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@@
   (paper "A4")
   (title_block
-    (date "2023-10-04")
+    (title "KiCad 2023 Asia Badge")
+    (date "2023-10-07")
     (rev "2")
+    (company "Beijing Exponential Deep Space")
   )
   (wire (pts (xy 119.38 78.74) (xy 110.49 78.74))
