File: hw/Buck_DCDC.kicad_sch (KiCad schematic)
At the start: 7 parts, among them U4 SY8088IAAC

Commit message: filled in LCSC
Parts:
- C10, C11: LCSC C15850 -> CA0134917
- C15: LCSC (none) -> CA0174301
- U4: LCSC (none) -> IC0444764; Vendor Model (none) -> SY8088IAAC
Changed lines of the file:
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@@
+      (effects (font (size 1.27 1.27)) hide)
+    )
+    (property "LCSC" "IC0444764" (at 111.76 68.58 0)
+      (effects (font (size 1.27 1.27)) hide)
+    )
+    (property "Vendor Model" "SY8088IAAC" (at 111.76 68.58 0)
       (effects (font (size 1.27 1.27)) hide)
     )
@@
       (effects (font (size 1.27 1.27)) hide)
     )
+    (property "LCSC" "CA0174301" (at 165.1 71.12 0)
+      (effects (font (size 1.27 1.27)) hide)
+    )
     (pin "1")
     (pin "2")
@@
       (effects (font (size 1.27 1.27)) hide)
     )
-    (property "LCSC" "C15850" (at 78.74 73.66 0)
+    (property "LCSC" "CA0134917" (at 78.74 73.66 0)
       (effects (font (size 1.27 1.27)) hide)
     )
@@
       (effects (font (size 1.27 1.27)) hide)
     )
-    (property "LCSC" "C15850" (at 181.61 76.2 0)
-      (effects (font (size 1.27 1.27)) hide)
-    )
+    (property "LCSC" "CA0134917" (at 181.61 76.2 0)
+      (effects (font (size 1.27 1.27)) hide)
+    )
